Commit message: fixes for installation on new system

File: model/mybot.xacro (robot description, xacro)
@@ -182,5 +182,5 @@
       <origin xyz="0 0 0" rpy="0 0 0"/>
       <geometry>
-        <mesh filename="package://mybot_description/meshes/hokuyo.dae"/>
+	      <mesh filename="$(find inverted_pendulum_control)/model/meshes/hokuyo.dae"/>
       </geometry>
     </visual>
