Commit message: Migrate package to ROS2 Humble and improve launch/controller flow

File: model/macros.xacro (robot description, xacro)
@@ -56,14 +56,4 @@
       <joint_properties damping="0.0" friction="0.0"/>
     </joint>
-    <transmission name="${lr}_trans">
-      <type>transmission_interface/SimpleTransmission</type>
-      <joint name="${lr}_wheel_hinge">
-        <hardwareInterface>EffortJointInterface</hardwareInterface>
-      </joint>
-      <actuator name="${lr}Motor">
-        <hardwareInterface>EffortJointInterface</hardwareInterface>
-        <mechanicalReduction>10</mechanicalReduction>
-      </actuator>
-    </transmission>
   </macro-->
 </robot>
